File: proyecto_arduino_ucc.kicad_sch (KiCad schematic)
At the start: 14 parts, among them J1 USB_A, J2 Header, U1 ATtiny85-20S

Commit message: Add files via upload
Other:
- moved on the sheet: R1, R4
Changed lines of the file:
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@@
-	)
-	(junction
-		(at 82.55 69.85)
-		(diameter 0)
-		(color 0 0 0 0)
-	)
-	(junction
-		(at 93.98 87.63)
-		(diameter 0)
-		(color 0 0 0 0)
 	)
 	(junction
@@
 	)
 	(junction
-		(at 142.24 60.96)
+		(at 92.71 87.63)
 		(diameter 0)
 		(color 0 0 0 0)
@@
 	)
 	(junction
-		(at 176.53 68.58)
-		(diameter 0)
-		(color 0 0 0 0)
-	)
-	(junction
 		(at 90.17 96.52)
 		(diameter 0)
@@
 	)
 	(junction
-		(at 175.26 68.58)
-		(diameter 0)
-		(color 0 0 0 0)
-	)
-	(junction
 		(at 95.25 85.09)
 		(diameter 0)
@@
 	(wire
 		(pts
-			(xy 142.24 60.96) (xy 142.24 62.23)
-		)
-		(stroke
-			(width 0)
-			(type default)
-		)
-	)
-	(wire
-		(pts
 			(xy 68.58 81.28) (xy 68.58 80.01)
 		)
@@
 	(wire
 		(pts
-			(xy 93.98 74.93) (xy 93.98 87.63)
+			(xy 92.71 74.93) (xy 92.71 87.63)
 		)
 		(stroke
@@
 	(wire
 		(pts
-			(xy 175.26 68.58) (xy 176.53 68.58)
-		)
-		(stroke
-			(width 0)
-			(type default)
-		)
-	)
-	(wire
-		(pts
-			(xy 168.91 68.58) (xy 175.26 68.58)
-		)
-		(stroke
-			(width 0)
-			(type default)
-		)
-	)
-	(wire
-		(pts
 			(xy 132.08 107.95) (xy 161.29 107.95)
 		)
@@
 	(wire
 		(pts
-			(xy 176.53 68.58) (xy 177.8 68.58)
+			(xy 92.71 87.63) (xy 104.14 87.63)
 		)
 		(stroke
@@
 	(wire
 		(pts
-			(xy 85.09 87.63) (xy 93.98 87.63)
+			(xy 85.09 87.63) (xy 92.71 87.63)
 		)
 		(stroke
@@
 	(wire
 		(pts
-			(xy 93.98 87.63) (xy 104.14 87.63)
-		)
-		(stroke
-			(width 0)
-			(type default)
-		)
-	)
-	(wire
-		(pts
 			(xy 134.62 58.42) (xy 134.62 68.58)
 		)
@@
 	(wire
 		(pts
-			(xy 176.53 68.58) (xy 176.53 69.85)
-		)
-		(stroke
-			(width 0)
-			(type default)
-		)
-	)
-	(wire
-		(pts
 			(xy 176.53 91.44) (xy 176.53 95.25)
 		)
@@
 	(wire
 		(pts
-			(xy 87.63 67.31) (xy 93.98 67.31)
+			(xy 87.63 67.31) (xy 92.71 67.31)
 		)
 		(stroke
@@
 	(wire
 		(pts
+			(xy 82.55 67.31) (xy 82.55 69.85)
+		)
+		(stroke
+			(width 0)
+			(type default)
+		)
+	)
+	(wire
+		(pts
 			(xy 161.29 68.58) (xy 134.62 68.58)
 		)
@@
 	(wire
 		(pts
-			(xy 182.88 68.58) (xy 193.04 68.58)
+			(xy 186.69 68.58) (xy 193.04 68.58)
 		)
 		(stroke
@@
 	(wire
 		(pts
+			(xy 168.91 68.58) (xy 179.07 68.58)
+		)
+		(stroke
+			(width 0)
+			(type default)
+		)
+	)
+	(wire
+		(pts
 			(xy 223.52 107.95) (xy 223.52 111.76)
 		)
@@
 	(wire
 		(pts
-			(xy 82.55 69.85) (xy 82.55 67.31)
-		)
-		(stroke
-			(width 0)
-			(type default)
-		)
-	)
-	(wire
-		(pts
 			(xy 71.12 87.63) (xy 85.09 87.63)
 		)
@@
 		(pts
 			(xy 71.12 87.63) (xy 71.12 85.09)
-		)
-		(stroke
-			(width 0)
-			(type default)
-		)
-	)
-	(wire
-		(pts
-			(xy 82.55 69.85) (xy 82.55 71.12)
 		)
 		(stroke
@@
 	(symbol
 		(lib_id "Device:R")
-		(at 93.98 71.12 0)
+		(at 92.71 71.12 0)
 		(unit 1)
 		(exclude_from_sim no)
@@
 		(fields_autoplaced yes)
 		(property "Reference" "R1"
-			(at 96.52 69.8499 0)
+			(at 95.25 69.8499 0)
 			(effects
 				(font
@@
 		)
 		(property "Value" "1.5K 5% 1/8W"
-			(at 96.52 72.3899 0)
+			(at 95.25 72.3899 0)
 			(effects
 				(font
@@
 		)
 		(property "Footprint" "Resistor_SMD:R_0805_2012Metric_Pad1.20x1.40mm_HandSolder"
-			(at 92.202 71.12 90)
+			(at 90.932 71.12 90)
 			(effects
 				(font
@@
 		)
 		(property "Datasheet" "~"
-			(at 93.98 71.12 0)
+			(at 92.71 71.12 0)
 			(effects
 				(font
@@
 		)
 		(property "Description" "Resistor"
-			(at 93.98 71.12 0)
+			(at 92.71 71.12 0)
 			(effects
 				(font
@@
 	(symbol
 		(lib_id "Device:R")
-		(at 179.07 68.58 90)
+		(at 182.88 68.58 90)
 		(unit 1)
 		(exclude_from_sim no)
@@
 		(fields_autoplaced yes)
 		(property "Reference" "R4"
-			(at 179.07 62.23 90)
+			(at 182.88 62.23 90)
 			(effects
 				(font
@@
 		)
 		(property "Value" "330 5% 1/8W"
-			(at 179.07 64.77 90)
+			(at 182.88 64.77 90)
 			(effects
 				(font
@@
 		)
 		(property "Footprint" "Resistor_SMD:R_0805_2012Metric_Pad1.20x1.40mm_HandSolder"
-			(at 179.07 70.358 90)
+			(at 182.88 70.358 90)
 			(effects
 				(font
@@
 		)
 		(property "Datasheet" "~"
-			(at 179.07 68.58 0)
+			(at 182.88 68.58 0)
 			(effects
 				(font
@@
 		)
 		(property "Description" "Resistor"
-			(at 179.07 68.58 0)
-			(effects
-				(font
+			(at 182.88 68.58 0)
+			(effects
+				(font

Commit message: Add files via upload
Connections:
- no-connect marks 0 -> 3
Changed lines of the file:
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@@
 	)
 	(junction
-		(at 71.12 85.09)
+		(at 82.55 80.01)
 		(diameter 0)
 		(color 0 0 0 0)
 	)
 	(junction
-		(at 71.12 87.63)
+		(at 95.25 85.09)
+		(diameter 0)
+		(color 0 0 0 0)
+	)
+	(junction
+		(at 129.54 87.63)
+		(diameter 0)
+		(color 0 0 0 0)
+	)
+	(junction
+		(at 87.63 67.31)
+		(diameter 0)
+		(color 0 0 0 0)
+	)
+	(junction
+		(at 92.71 87.63)
+		(diameter 0)
+		(color 0 0 0 0)
+	)
+	(junction
+		(at 92.71 85.09)
 		(diameter 0)
 		(color 0 0 0 0)
@@
 	)
 	(junction
-		(at 129.54 87.63)
-		(diameter 0)
-		(color 0 0 0 0)
-	)
-	(junction
-		(at 87.63 67.31)
-		(diameter 0)
-		(color 0 0 0 0)
-	)
-	(junction
-		(at 92.71 87.63)
-		(diameter 0)
-		(color 0 0 0 0)
-	)
-	(junction
-		(at 71.12 80.01)
-		(diameter 0)
-		(color 0 0 0 0)
-	)
-	(junction
 		(at 90.17 96.52)
 		(diameter 0)
@@
 		(color 0 0 0 0)
 	)
-	(junction
-		(at 95.25 85.09)
-		(diameter 0)
-		(color 0 0 0 0)
-	)
-	(wire
-		(pts
-			(xy 68.58 81.28) (xy 68.58 80.01)
-		)
-		(stroke
-			(width 0)
-			(type default)
-		)
-	)
-	(wire
-		(pts
-			(xy 92.71 74.93) (xy 92.71 87.63)
-		)
-		(stroke
-			(width 0)
-			(type default)
-		)
-	)
-	(wire
-		(pts
-			(xy 64.77 85.09) (xy 71.12 85.09)
-		)
-		(stroke
-			(width 0)
-			(type default)
-		)
-	)
-	(wire
-		(pts
-			(xy 64.77 86.36) (xy 64.77 85.09)
+	(no_connect
+		(at 60.96 95.25)
+	)
+	(no_connect
+		(at 121.92 58.42)
+	)
+	(no_connect
+		(at 139.7 58.42)
+	)
+	(wire
+		(pts
+			(xy 92.71 85.09) (xy 95.25 85.09)
+		)
+		(stroke
+			(width 0)
+			(type default)
+		)
+	)
+	(wire
+		(pts
+			(xy 92.71 74.93) (xy 92.71 85.09)
 		)
 		(stroke
@@
 	(wire
 		(pts
+			(xy 95.25 85.09) (xy 113.03 85.09)
+		)
+		(stroke
+			(width 0)
+			(type default)
+		)
+	)
+	(wire
+		(pts
 			(xy 137.16 58.42) (xy 137.16 102.87)
 		)
@@
 	(wire
 		(pts
-			(xy 95.25 85.09) (xy 113.03 85.09)
+			(xy 92.71 85.09) (xy 92.71 87.63)
 		)
 		(stroke
@@
 	(wire
 		(pts
-			(xy 71.12 85.09) (xy 95.25 85.09)
-		)
-		(stroke
-			(width 0)
-			(type default)
-		)
-	)
-	(wire
-		(pts
 			(xy 92.71 87.63) (xy 104.14 87.63)
 		)
@@
 	(wire
 		(pts
+			(xy 71.12 87.63) (xy 85.09 87.63)
+		)
+		(stroke
+			(width 0)
+			(type default)
+		)
+	)
+	(wire
+		(pts
 			(xy 134.62 58.42) (xy 134.62 68.58)
 		)
@@
 	(wire
 		(pts
+			(xy 71.12 80.01) (xy 82.55 80.01)
+		)
+		(stroke
+			(width 0)
+			(type default)
+		)
+	)
+	(wire
+		(pts
 			(xy 90.17 96.52) (xy 95.25 96.52)
 		)
@@
 	(wire
 		(pts
-			(xy 71.12 80.01) (xy 82.55 80.01)
-		)
-		(stroke
-			(width 0)
-			(type default)
-		)
-	)
-	(wire
-		(pts
-			(xy 68.58 80.01) (xy 71.12 80.01)
-		)
-		(stroke
-			(width 0)
-			(type default)
-		)
-	)
-	(wire
-		(pts
 			(xy 186.69 68.58) (xy 193.04 68.58)
 		)
@@
 	(wire
 		(pts
-			(xy 71.12 87.63) (xy 85.09 87.63)
+			(xy 71.12 85.09) (xy 92.71 85.09)
 		)
 		(stroke
@@
 		(pts
 			(xy 129.54 58.42) (xy 129.54 87.63)
-		)
-		(stroke
-			(width 0)
-			(type default)
-		)
-	)
-	(wire
-		(pts
-			(xy 71.12 87.63) (xy 71.12 85.09)
 		)
 		(stroke
@@
 					(unit 1)
 				)
+			)
+		)
+	)
+	(symbol
+		(lib_id "power:PWR_FLAG")
+		(at 82.55 80.01 180)
+		(unit 1)
+		(exclude_from_sim no)
+		(in_bom yes)
+		(on_board yes)
+		(dnp no)
+		(property "Reference" "#FLG03"
+			(at 82.55 81.915 0)
+			(effects
+				(font
+					(size 1.27 1.27)
+				)
+				(hide yes)
+			)
+		)
+		(property "Value" "PWR_FLAG"
+			(at 82.804 83.566 0)
+			(effects
+				(font
+					(size 1.27 1.27)
+				)
+			)
+		)
+		(property "Footprint" ""
+			(at 82.55 80.01 0)
+			(effects
+				(font
+					(size 1.27 1.27)
+				)
+				(hide yes)
+			)
+		)
+		(property "Datasheet" "~"
+			(at 82.55 80.01 0)
+			(effects
+				(font
+					(size 1.27 1.27)
+				)
+				(hide yes)
+			)
+		)
+		(property "Description" "Special symbol for telling ERC where power comes from"
+			(at 82.55 80.01 0)
+			(effects
+				(font
+					(size 1.27 1.27)
+				)
+				(hide yes)
+			)
+		)
+		(pin "1"
+		)
+		(instances
+			(project ""
+				(path "/ff8fc11e-9292-42bc-9b99-842903e65f08"
+					(reference "#FLG03")
+					(unit 1)
+				)
